Commit message: fix transparent fingers; fix fingers offset from the base

File: wsg_50_simulation/urdf/wsg_50.urdf.xacro (robot description, xacro)
@@ -54,5 +54,5 @@
   </link>
   <!-- GRIPPER LEFT -->
-  <joint name="${name}_finger_left_joint" type="prismatic">
+  <joint name="${name}_finger_left_joint" type="fixed">
      <limit lower="-0.055" upper="-0.0027" effort="1.0" velocity="1.0"/>
      <origin xyz="0 0 0" rpy="0 0 0" />      <!--origin xyz="-0.0067 0 0.049" rpy="0 0 0" /-->
@@ -83,6 +83,6 @@
 	     <!--box size="0.0175 0.03 0.024"/-->
           </geometry>
-          <material name="black">
-		<color rgba="0 0 0 0"/>
+          <material name="white">
+		<color rgba="1 1 1 1"/>
       	  </material>
       </visual>
@@ -102,5 +102,5 @@
   <!-- LEFT FINGER -->
   <joint name="${name}_guide_joint_finger_left" type="fixed">
-     <origin xyz="${finger_tip} 0 ${finger_length}" rpy="0 0 0" />
+     <origin xyz="${-finger_tip} 0 0" rpy="0 0 0" />
      <parent link="${name}_gripper_left"/>
      <child link="${name}_finger_left" />
@@ -122,6 +122,6 @@
              <mesh filename="package://wsg_50_simulation/meshes/WSG-FMF.stl" scale="0.001 0.001 0.001"/>
           </geometry>
-          <material name="black">
-		<color rgba="0 0 0 0"/>
+          <material name="white">
+		<color rgba="1 1 1 1"/>
       	  </material>
       </visual>
@@ -139,5 +139,5 @@
   </gazebo>
   <!-- GRIPPER RIGHT -->
-  <joint name="${name}_finger_right_joint" type="prismatic">
+  <joint name="${name}_finger_right_joint" type="fixed">
      <limit lower="0.0027" upper="0.055" effort="1.0" velocity="1.0"/>
      <origin xyz="0 0 0" rpy="0 0 3.14159" />
@@ -168,6 +168,6 @@
 	     <!--box size="0.0175 0.03 0.024"/-->
           </geometry>
-          <material name="black">
-		<color rgba="0 0 0 0"/>
+          <material name="white">
+		<color rgba="1 1 1 1"/>
       	  </material>
       </visual>
@@ -187,5 +187,5 @@
   <!-- RIGHT FINGER -->
   <joint name="${name}_guide_joint_finger_right" type="fixed">
-     <origin xyz="${finger_tip} 0 ${finger_length}" rpy="0 0 0" />
+     <origin xyz="${-finger_tip} 0 0" rpy="0 0 0" />
      <parent link="${name}_gripper_right"/>
      <child link="${name}_finger_right" />
@@ -207,6 +207,6 @@
              <mesh filename="package://wsg_50_simulation/meshes/WSG-FMF.stl" scale="0.001 0.001 0.001"/>
           </geometry>
-          <material name="black">
-		<color rgba="0 0 0 0"/>
+          <material name="white">
+		<color rgba="1 1 1 1"/>
       	  </material>
       </visual>
